Commit message: Stuff for working with new ROS kinova

File: jaco_control/urdf/jaco_arm.urdf (robot description, URDF)
Before this commit: robot jaco, 12 links, 11 joints
Links:
- removed link jaco_link_1
- removed link jaco_link_2
- removed link jaco_link_3
- removed link jaco_link_4
- removed link jaco_link_5
- removed link jaco_link_base
- removed link jaco_link_finger_1
- removed link jaco_link_finger_2
- removed link jaco_link_finger_3
- removed link jaco_link_hand
- removed link jaco_link_tool
- added link j2n6s300_end_effector; collision box size=0 0 0; visual box size=0 0 0
- added link j2n6s300_link_1, mass 0.7477; collision mesh filename=package://kinova_description/meshes/shoulder.dae; visual mesh filename=package://kinova_description/meshes/ring_big.STL
- added link j2n6s300_link_2, mass 0.99; collision mesh filename=package://kinova_description/meshes/arm.dae; visual mesh filename=package://kinova_description/meshes/arm.dae
- added link j2n6s300_link_3, mass 0.6763; collision mesh filename=package://kinova_description/meshes/forearm.dae; visual mesh filename=package://kinova_description/meshes/forearm.dae
- added link j2n6s300_link_4, mass 0.1785; collision mesh filename=package://kinova_description/meshes/wrist.dae; visual mesh filename=package://kinova_description/meshes/ring_small.STL
- added link j2n6s300_link_5, mass 0.1785; collision mesh filename=package://kinova_description/meshes/wrist.dae; visual mesh filename=package://kinova_description/meshes/ring_small.STL
- added link j2n6s300_link_6, mass 0.727; collision mesh filename=package://kinova_description/meshes/hand_3finger.dae; visual mesh filename=package://kinova_description/meshes/hand_3finger.dae
- added link j2n6s300_link_base, mass 0.46784; collision mesh filename=package://kinova_description/meshes/base.dae; visual mesh filename=package://kinova_description/meshes/base.dae
- added link j2n6s300_link_finger_1, mass 0.01; collision mesh filename=package://kinova_description/meshes/finger_proximal.dae; visual mesh filename=package://kinova_description/meshes/finger_proximal.dae
- added link j2n6s300_link_finger_2, mass 0.01; collision mesh filename=package://kinova_description/meshes/finger_proximal.dae; visual mesh filename=package://kinova_description/meshes/finger_proximal.dae
- added link j2n6s300_link_finger_3, mass 0.01; collision mesh filename=package://kinova_description/meshes/finger_proximal.dae; visual mesh filename=package://kinova_description/meshes/finger_proximal.dae
- added link j2n6s300_link_finger_tip_1, mass 0.01; collision mesh filename=package://kinova_description/meshes/finger_distal.dae; visual mesh filename=package://kinova_description/meshes/finger_distal.dae
- added link j2n6s300_link_finger_tip_2, mass 0.01; collision mesh filename=package://kinova_description/meshes/finger_distal.dae; visual mesh filename=package://kinova_description/meshes/finger_distal.dae
- added link j2n6s300_link_finger_tip_3, mass 0.01; collision mesh filename=package://kinova_description/meshes/finger_distal.dae; visual mesh filename=package://kinova_description/meshes/finger_distal.dae
- added link world
Joints:
- removed joint jaco_joint_1
- removed joint jaco_joint_2
- removed joint jaco_joint_3
- removed joint jaco_joint_4
- removed joint jaco_joint_5
- removed joint jaco_joint_6
- removed joint jaco_joint_base
- removed joint jaco_joint_finger_1
- removed joint jaco_joint_finger_2
- removed joint jaco_joint_finger_3
- removed joint jaco_joint_tool
- added joint connect_root_and_world: type fixed, parent world, child root, origin xyz=0 0 0 rpy=0 0 0
- added joint j2n6s300_joint_1: type continuous, parent j2n6s300_link_base, child j2n6s300_link_1, origin xyz=0 0 0.15675 rpy=0 3.14159265359 0, axis 0 0 1, limit lower=-6.28318530718 upper=6.28318530718 effort=2000 velocity=1
- added joint j2n6s300_joint_2: type revolute, parent j2n6s300_link_1, child j2n6s300_link_2, origin xyz=0 0.0016 -0.11875 rpy=-1.57079632679 0 3.14159265359, axis 0 0 1, limit lower=0.523598775598 upper=5.75958653158 effort=2000 velocity=1
- added joint j2n6s300_joint_3: type revolute, parent j2n6s300_link_2, child j2n6s300_link_3, origin xyz=0 -0.410 0 rpy=0 3.14159265359 0, axis 0 0 1, limit lower=0.523598775598 upper=5.75958653158 effort=2000 velocity=1
- added joint j2n6s300_joint_4: type continuous, parent j2n6s300_link_3, child j2n6s300_link_4, origin xyz=0 0.2073 -0.0114 rpy=-1.57079632679 0 3.14159265359, axis 0 0 1, limit lower=-6.28318530718 upper=6.28318530718 effort=2000 velocity=1
- added joint j2n6s300_joint_5: type continuous, parent j2n6s300_link_4, child j2n6s300_link_5, origin xyz=0 -0.03703 -0.06414 rpy=1.0471975512 0 3.14159265359, axis 0 0 1, limit lower=-6.28318530718 upper=6.28318530718 effort=2000 velocity=1
- added joint j2n6s300_joint_6: type continuous, parent j2n6s300_link_5, child j2n6s300_link_6, origin xyz=0 -0.03703 -0.06414 rpy=1.0471975512 0 3.14159265359, axis 0 0 1, limit lower=-6.28318530718 upper=6.28318530718 effort=2000 velocity=1
- added joint j2n6s300_joint_base: type fixed, parent root, child j2n6s300_link_base, origin xyz=0 0 0 rpy=0 0 0, axis 0 0 0, limit lower=0 upper=0 effort=2000 velocity=1
- added joint j2n6s300_joint_end_effector: type fixed, parent j2n6s300_link_6, child j2n6s300_end_effector, origin xyz=0 0 -0.1600 rpy=3.14159265359 0 0, axis 0 0 0, limit lower=0 upper=0 effort=2000 velocity=1
- added joint j2n6s300_joint_finger_1: type revolute, parent j2n6s300_link_6, child j2n6s300_link_finger_1, origin xyz=0.00279 0.03126 -0.11467 rpy=-1.570796327 .649262481663582 1.35961148639407, axis 0 0 1, limit lower=0 upper=2 effort=2000 velocity=1
- added joint j2n6s300_joint_finger_2: type revolute, parent j2n6s300_link_6, child j2n6s300_link_finger_2, origin xyz=0.02226 -0.02707 -0.11482 rpy=-1.570796327 .649262481663582 -1.38614049188413, axis 0 0 1, limit lower=0 upper=2 effort=2000 velocity=1
- added joint j2n6s300_joint_finger_3: type revolute, parent j2n6s300_link_6, child j2n6s300_link_finger_3, origin xyz=-0.02226 -0.02707 -0.11482 rpy=-1.570796327 .649262481663582 -1.75545216211587, axis 0 0 1, limit lower=0 upper=2 effort=2000 velocity=1
- added joint j2n6s300_joint_finger_tip_1: type fixed, parent j2n6s300_link_finger_1, child j2n6s300_link_finger_tip_1, origin xyz=0.044 -0.003 0 rpy=0 0 0, axis 0 0 1, limit lower=0 upper=2 effort=2000 velocity=1
- added joint j2n6s300_joint_finger_tip_2: type fixed, parent j2n6s300_link_finger_2, child j2n6s300_link_finger_tip_2, origin xyz=0.044 -0.003 0 rpy=0 0 0, axis 0 0 1, limit lower=0 upper=2 effort=2000 velocity=1
- added joint j2n6s300_joint_finger_tip_3: type fixed, parent j2n6s300_link_finger_3, child j2n6s300_link_finger_tip_3, origin xyz=0.044 -0.003 0 rpy=0 0 0, axis 0 0 1, limit lower=0 upper=2 effort=2000 velocity=1
